Commit message: updated robot

File: go_chase_it/my_robot/urdf/my_robot.xacro (robot description, xacro)
@@ -2,4 +2,6 @@
 <robot name="my_robot" xmlns:xacro="http://www.ros.org/wiki/xacro">
   <xacro:include filename="$(find my_robot)/urdf/my_robot.gazebo" />
+  <xacro:property name="wheel_radius" value="0.15" />
+  <xacro:property name="wheel_length" value="0.05" />
   <link name="robot_footprint"></link>
   <joint name="robot_footprint_joint" type="fixed">
@@ -12,5 +14,5 @@
     <inertial>
       <mass value="15.0"/>
-      <origin xyz="0.0 0 0" rpy=" 0 0 0"/>
+      <origin xyz="-0.1 0 0" rpy=" 0 0 0"/>
       <inertia
           ixx="0.1" ixy="0" ixz="0"
@@ -31,14 +33,14 @@
       </geometry>
     </visual>
-    <collision name='back_caster_collision'>
-      <origin xyz="-0.15 0 -0.05" rpy=" 0 0 0"/>
+    <collision name='upper_box_collision'>
+      <origin xyz="-0.1 0 .1" rpy=" 0 0 0"/>
       <geometry>
-        <sphere radius="0.0499"/>
+        <box size=".2 .2 .2"/>
       </geometry>
     </collision>
-    <visual name='back_caster_visual'>
-      <origin xyz="-0.15 0 -0.05" rpy=" 0 0 0"/>
+    <visual>
+      <origin xyz="-0.1 0 .1" rpy=" 0 0 0"/>
       <geometry>
-        <sphere radius="0.05"/>
+        <box size=".2 .2 .2"/>
       </geometry>
     </visual>
@@ -60,5 +62,5 @@
       <origin xyz="0 0 0" rpy=" 0 1.5707 1.5707"/>
       <geometry>
-        <cylinder radius="0.1" length="0.05"/>
+        <cylinder radius="0.15" length="0.05"/>
       </geometry>
     </collision>
@@ -66,5 +68,5 @@
       <origin xyz="0 0 0" rpy=" 0 1.5707 1.5707"/>
       <geometry>
-        <cylinder radius="0.1" length="0.05"/>
+	<cylinder radius="${wheel_radius}" length="${wheel_length}"/>
       </geometry>
     </visual>
@@ -83,11 +85,11 @@
       <origin xyz="0 0 0" rpy=" 0 1.5707 1.5707"/>
       <geometry>
-        <cylinder radius="0.1" length="0.05"/>
+	<cylinder radius="${wheel_radius}" length="${wheel_length}"/>
       </geometry>
     </collision>
-    <visual name='right_wheel_visual'>
+    <visual>
       <origin xyz="0 0 0" rpy=" 0 1.5707 1.5707"/>
       <geometry>
-        <cylinder radius="0.1" length="0.05"/>
+        <cylinder radius="0.15" length="0.05"/>
       </geometry>
     </visual>
@@ -103,5 +105,5 @@
   </link>
   <joint type="continuous" name="left_wheel_hinge">
-    <origin xyz="0 0.15 0" rpy="0 0 0"/>
+    <origin xyz="-0.15 0.15 0.05" rpy="0 0 0"/>
     <child link="left_wheel"/>
     <parent link="chassis"/>
@@ -111,5 +113,5 @@
   </joint>
   <joint type="continuous" name="right_wheel_hinge">
-    <origin xyz="0 -0.15 0" rpy="0 0 0"/>
+    <origin xyz="-0.15 -0.15 0.05" rpy="0 0 0"/>
     <child link="right_wheel"/>
     <parent link="chassis"/>
@@ -129,5 +131,5 @@
     </inertial>
     <visual name='camera_visual'>
-      <origin xyz="0 0 0" rpy="0 0 0"/>
+      <origin xyz="-.2 0 .1" rpy="0 0 0"/>
       <geometry>
         <box size=".05 .05 .05"/>
@@ -158,5 +160,5 @@
     </inertial>
     <visual name='hokuyo_visual'>
-      <origin xyz="0 0 0" rpy="0 0 0"/>
+      <origin xyz="-0.2 0 0.1" rpy="0 0 0"/>
       <geometry>
         <mesh filename="package://my_robot/meshes/hokuyo.dae"/>
@@ -176,3 +178,15 @@
     <axis xyz="0 1 0"/>
   </joint>
+  <gazebo reference="left_wheel">
+     <material>Gazebo/Black</material>
+  </gazebo>
+  <gazebo reference="right_wheel">
+     <material>Gazebo/Black</material>
+  </gazebo>
+  <gazebo reference="camera">
+     <material>Gazebo/Blue</material>
+  </gazebo>
+  <gazebo reference="chassis">
+     <material>Gazebo/Yellow</material>
+  </gazebo>
 </robot>
